File: V4N4AG0RTH0N.kicad_pcb (KiCad board)
At the start: 2 copper layers, 77.8 x 38.1 mm, 24 parts, among them SW1 SW_Push, U1 ATmega32U4-A, Y1 16MHz

Commit message: Almost done?
Parts:
- added D10: SOD-123, Diode_SMD:D_SOD-123, B.Cu at (94.0, 63.4)
- added D11: SOD-123, Diode_SMD:D_SOD-123, B.Cu at (113.0, 63.4)
- added D12: SOD-123, Diode_SMD:D_SOD-123, B.Cu at (132.1, 63.4)
- added D13: SOD-123, Diode_SMD:D_SOD-123, B.Cu at (165.1, 63.4)
- added D14: SOD-123, Diode_SMD:D_SOD-123, B.Cu at (184.2, 63.4)
- added D15: SOD-123, Diode_SMD:D_SOD-123, B.Cu at (203.2, 63.4)
- added D16: SOD-123, Diode_SMD:D_SOD-123, B.Cu at (222.2, 63.4)
- added D17: SOD-123, Diode_SMD:D_SOD-123, B.Cu at (241.3, 63.4)
- added D18: SOD-123, Diode_SMD:D_SOD-123, B.Cu at (260.3, 63.4)
- added D19: SOD-123, Diode_SMD:D_SOD-123, B.Cu at (36.8, 82.4)
- added D20: SOD-123, Diode_SMD:D_SOD-123, B.Cu at (55.9, 82.4)
- added D21: SOD-123, Diode_SMD:D_SOD-123, B.Cu at (74.9, 82.4)
- added D22: SOD-123, Diode_SMD:D_SOD-123, B.Cu at (94.0, 82.4)
- added D23: SOD-123, Diode_SMD:D_SOD-123, B.Cu at (113.0, 82.4)
- added D24: SOD-123, Diode_SMD:D_SOD-123, B.Cu at (132.1, 82.4)
- added D25: SOD-123, Diode_SMD:D_SOD-123, B.Cu at (165.1, 82.4)
- added D26: SOD-123, Diode_SMD:D_SOD-123, B.Cu at (184.2, 82.4)
- added D27: SOD-123, Diode_SMD:D_SOD-123, B.Cu at (203.2, 82.4)
- added D28: SOD-123, Diode_SMD:D_SOD-123, B.Cu at (222.2, 82.4)
- added D29: SOD-123, Diode_SMD:D_SOD-123, B.Cu at (241.3, 82.4)
- added D30: SOD-123, Diode_SMD:D_SOD-123, B.Cu at (260.4, 82.4)
- added D31: SOD-123, Diode_SMD:D_SOD-123, B.Cu at (36.8, 101.5)
- added D32: SOD-123, Diode_SMD:D_SOD-123, B.Cu at (55.9, 101.5)
- added D33: SOD-123, Diode_SMD:D_SOD-123, B.Cu at (74.9, 101.5)
- added D34: SOD-123, Diode_SMD:D_SOD-123, B.Cu at (98.8, 101.5)
- added D35: SOD-123, Diode_SMD:D_SOD-123, B.Cu at (113.0, 101.5)
- added D36: SOD-123, Diode_SMD:D_SOD-123, B.Cu at (136.9, 101.5)
- added D37: SOD-123, Diode_SMD:D_SOD-123, B.Cu at (170.2, 101.5)
- added D38: SOD-123, Diode_SMD:D_SOD-123, B.Cu at (184.2, 101.5)
- added D39: SOD-123, Diode_SMD:D_SOD-123, B.Cu at (208.3, 101.5)
- added D40: SOD-123, Diode_SMD:D_SOD-123, B.Cu at (222.2, 101.5)
- added D41: SOD-123, Diode_SMD:D_SOD-123, B.Cu at (241.3, 101.5)
- added D42: SOD-123, Diode_SMD:D_SOD-123, B.Cu at (260.4, 101.5)
- added D43: SOD-123, Diode_SMD:D_SOD-123, B.Cu at (36.8, 120.5)
- added D44: SOD-123, Diode_SMD:D_SOD-123, B.Cu at (55.9, 120.5)
- added D45: SOD-123, Diode_SMD:D_SOD-123, B.Cu at (74.9, 120.5)
- added D46: SOD-123, Diode_SMD:D_SOD-123, B.Cu at (113.0, 120.5)
- added D47: SOD-123, Diode_SMD:D_SOD-123, B.Cu at (184.2, 120.5)
- added D48: SOD-123, Diode_SMD:D_SOD-123, B.Cu at (222.2, 120.5)
- added D49: SOD-123, Diode_SMD:D_SOD-123, B.Cu at (241.3, 120.5)
- added D5: SOD-123, Diode_SMD:D_SOD-123, B.Cu at (121.9, 44.3)
- added D50: SOD-123, Diode_SMD:D_SOD-123, B.Cu at (260.4, 120.5)
- added D51: LED, LED_THT:LED_D3.0mm, F.Cu at (27.4, 31.5)
- added D52: LED, LED_THT:LED_D3.0mm, F.Cu at (27.4, 37.5)
- added D53: LED, LED_THT:LED_D3.0mm, F.Cu at (27.4, 43.4)
- added D6: SOD-123, Diode_SMD:D_SOD-123, B.Cu at (141.0, 44.3)
- added D7: SOD-123, Diode_SMD:D_SOD-123, B.Cu at (36.8, 63.4)
- added D8: SOD-123, Diode_SMD:D_SOD-123, B.Cu at (55.9, 63.4)
- added D9: SOD-123, Diode_SMD:D_SOD-123, B.Cu at (74.9, 63.4)
- added F2: Polyfuse_Small, Fuse:Fuse_1206_3216Metric, F.Cu at (111.4, 11.2)
- added MX10: MX-NoLED, MX_Alps_Hybrid:MX-1U-NoLED, F.Cu at (90.5, 57.1)
- added MX11: MX-NoLED, MX_Alps_Hybrid:MX-1U-NoLED, F.Cu at (109.5, 57.1)
- added MX12: MX-NoLED, MX_Alps_Hybrid:MX-1U-NoLED, F.Cu at (128.6, 57.1)
- added MX13: MX-NoLED, MX_Alps_Hybrid:MX-1U-NoLED, F.Cu at (161.9, 57.1)
- added MX14: MX-NoLED, MX_Alps_Hybrid:MX-1U-NoLED, F.Cu at (181.0, 57.1)
- added MX15: MX-NoLED, MX_Alps_Hybrid:MX-1U-NoLED, F.Cu at (200.0, 57.1)
- added MX16: MX-NoLED, MX_Alps_Hybrid:MX-1U-NoLED, F.Cu at (219.1, 57.1)
- added MX17: MX-NoLED, MX_Alps_Hybrid:MX-1U-NoLED, F.Cu at (238.1, 57.1)
- added MX18: MX-NoLED, MX_Alps_Hybrid:MX-1U-NoLED, F.Cu at (257.2, 57.1)
- added MX19: MX-NoLED, MX_Alps_Hybrid:MX-1U-NoLED, F.Cu at (33.3, 76.2)
- added MX20: MX-NoLED, MX_Alps_Hybrid:MX-1U-NoLED, F.Cu at (52.4, 76.2)
- added MX21: MX-NoLED, MX_Alps_Hybrid:MX-1U-NoLED, F.Cu at (71.4, 76.2)
- added MX22: MX-NoLED, MX_Alps_Hybrid:MX-1U-NoLED, F.Cu at (90.5, 76.2)
- added MX23: MX-NoLED, MX_Alps_Hybrid:MX-1U-NoLED, F.Cu at (109.5, 76.2)
- added MX24: MX-NoLED, MX_Alps_Hybrid:MX-1U-NoLED, F.Cu at (128.6, 76.2)
- added MX25: MX-NoLED, MX_Alps_Hybrid:MX-1U-NoLED, F.Cu at (161.9, 76.2)
- added MX26: MX-NoLED, MX_Alps_Hybrid:MX-1U-NoLED, F.Cu at (181.0, 76.2)
- added MX27: MX-NoLED, MX_Alps_Hybrid:MX-1U-NoLED, F.Cu at (200.0, 76.2)
- added MX28: MX-NoLED, MX_Alps_Hybrid:MX-1U-NoLED, F.Cu at (219.1, 76.2)
- added MX29: MX-NoLED, MX_Alps_Hybrid:MX-1U-NoLED, F.Cu at (238.1, 76.2)
- added MX30: MX-NoLED, MX_Alps_Hybrid:MX-1U-NoLED, F.Cu at (257.2, 76.2)
- added MX31: MX-NoLED, MX_Alps_Hybrid:MX-1U-NoLED, F.Cu at (33.3, 95.2)
- added MX32: MX-NoLED, MX_Alps_Hybrid:MX-1U-NoLED, F.Cu at (52.4, 95.2)
- added MX33: MX-NoLED, MX_Alps_Hybrid:MX-1U-NoLED, F.Cu at (71.4, 95.2)
- added MX34: MX-NoLED, MX_Alps_Hybrid:MX-1U-NoLED, F.Cu at (90.5, 95.2)
- added MX35: MX-NoLED, MX_Alps_Hybrid:MX-1U-NoLED, F.Cu at (109.5, 95.2)
- added MX36: MX-NoLED, MX_Alps_Hybrid:MX-1U-NoLED, F.Cu at (128.6, 95.2)
- added MX37: MX-NoLED, MX_Alps_Hybrid:MX-1U-NoLED, F.Cu at (161.9, 95.2)
- added MX38: MX-NoLED, MX_Alps_Hybrid:MX-1U-NoLED, F.Cu at (181.0, 95.2)
- added MX39: MX-NoLED, MX_Alps_Hybrid:MX-1U-NoLED, F.Cu at (200.0, 95.2)
- added MX40: MX-NoLED, MX_Alps_Hybrid:MX-1U-NoLED, F.Cu at (219.1, 95.2)
- added MX41: MX-NoLED, MX_Alps_Hybrid:MX-1U-NoLED, F.Cu at (238.1, 95.2)
- added MX42: MX-NoLED, MX_Alps_Hybrid:MX-1U-NoLED, F.Cu at (257.2, 95.2)
- added MX43: MX-NoLED, MX_Alps_Hybrid:MX-1U-NoLED, F.Cu at (33.3, 114.3)
- added MX44: MX-NoLED, MX_Alps_Hybrid:MX-1U-NoLED, F.Cu at (52.4, 114.3)
- added MX45: MX-NoLED, MX_Alps_Hybrid:MX-1U-NoLED, F.Cu at (71.4, 114.3)
- added MX46: MX-NoLED, MX_Alps_Hybrid:MX-3U-ReversedStabilizers-NoLED, F.Cu at (109.5, 114.3)
- added MX47: MX-NoLED, MX_Alps_Hybrid:MX-3U-ReversedStabilizers-NoLED, F.Cu at (181.0, 114.3)
- added MX48: MX-NoLED, MX_Alps_Hybrid:MX-1U-NoLED, F.Cu at (219.1, 114.3)
- added MX49: MX-NoLED, MX_Alps_Hybrid:MX-1U-NoLED, F.Cu at (238.1, 114.3)
- added MX5: MX-NoLED, MX_Alps_Hybrid:MX-1U-NoLED, F.Cu at (119.1, 38.1)
- added MX50: MX-NoLED, MX_Alps_Hybrid:MX-1U-NoLED, F.Cu at (257.2, 114.3)
- added MX6: MX-NoLED, MX_Alps_Hybrid:MX-1U-NoLED, F.Cu at (138.1, 38.1)
- added MX7: MX-NoLED, MX_Alps_Hybrid:MX-1U-NoLED, F.Cu at (33.3, 57.1)
- added MX8: MX-NoLED, MX_Alps_Hybrid:MX-1U-NoLED, F.Cu at (52.4, 57.1)
- added MX9: MX-NoLED, MX_Alps_Hybrid:MX-1U-NoLED, F.Cu at (71.4, 57.1)
- added R5: 330, Resistor_SMD:R_0805_2012Metric, F.Cu at (115.0, 17.3)
- added R6: 330, Resistor_SMD:R_0805_2012Metric, F.Cu at (120.6, 12.9)
- added R7: 330, Resistor_SMD:R_0805_2012Metric, F.Cu at (110.1, 24.4)
- added R8: 5.1K, Resistor_SMD:R_0805_2012Metric, F.Cu at (115.0, 20.3)
- added R9: 5.1K, Resistor_SMD:R_0805_2012Metric, F.Cu at (119.4, 17.2)
- C1, C2, C3, C4, C5, C6, C7, R1, R2, R3, R4, SW1, Y1: moved to F.Cu
- F1: value 500mA -> Polyfuse_Small; moved to F.Cu
- USB1: value Molex-0548190589 -> HRO-TYPE-C-31-M-12; footprint random-keyboard-parts:Molex-0548190589 -> Type-C:HRO-TYPE-C-31-M-12
- moved SW1 136.2 mm to (88.3, 21.6), turned to 0 degrees
- moved MX1 135.9 mm to (42.9, 38.1)
- moved MX2 135.9 mm to (61.9, 38.1)
- moved D1 135.1 mm to (45.7, 44.3)
- moved D2 135.1 mm to (64.8, 44.3)
- moved C2 134.4 mm to (106.1, 18.4), turned to 0 degrees
- moved C7 130.5 mm to (110.6, 18.4), turned to 0 degrees
- moved MX3 130.0 mm to (81.0, 38.1)
- moved MX4 130.0 mm to (100.0, 38.1)
- moved U1 129.6 mm to (73.7, 20.6)
- moved F1 128.4 mm to (106.7, 15.3), turned to 0 degrees
- moved C3 128.3 mm to (111.7, 14.3), turned to 0 degrees
- moved R4 127.9 mm to (110.1, 21.4), turned to 0 degrees
- moved D3 126.7 mm to (83.8, 44.3)
- moved D4 126.7 mm to (102.9, 44.3)
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Connections:
- D2 pad 1: ROW1 -> ROW0
- D4 pad 1: ROW1 -> ROW0
- MX2 pad 1: COL0 -> COL1
- MX3 pad 1: COL1 -> COL2
- MX4 pad 1: COL1 -> COL3
- U1 pad 26: COL0 -> Net-(U1-Pad26)
- U1 pad 27: COL1 -> Net-(U1-Pad27)
- U1 pad 28: ROW0 -> Net-(U1-Pad28)
- U1 pad 29: ROW1 -> Net-(U1-Pad29)
- U1 pad 39: Net-(U1-Pad39) -> LED_3
- U1 pad 40: Net-(U1-Pad40) -> LED_2
- U1 pad 41: Net-(U1-Pad41) -> LED_1
- USB1 pad 2: Net-(USB1-Pad2) -> VCC
- USB1 pad 3: D+ -> Net-(USB1-Pad3)
- USB1 pad 4: D- -> Net-(R8-Pad2)
- USB1 pad 5: VCC -> D-
- USB1 pad 6: Net-(USB1-Pad6) -> D+
Routing:
- net ROW4: track 0.00 -> 236.8 mm
- net ROW3: track 0.00 -> 223.5 mm
- net ROW2: track 0.00 -> 223.5 mm
- net ROW1: track 65.0 -> 223.5 mm, vias 2 -> 0
- net GND: track 110.2 -> 0.00 mm
- net COL2: track 0.00 -> 75.7 mm
- net COL4: track 0.00 -> 75.7 mm
- net COL5: track 0.00 -> 57.6 mm
- net COL3: track 0.00 -> 57.6 mm
- net COL9: track 0.00 -> 54.4 mm
- net COL7: track 0.00 -> 54.4 mm
- net COL11: track 0.00 -> 54.4 mm
- net COL10: track 0.00 -> 54.4 mm
- net ROW0: track 52.4 -> 95.2 mm, vias 3 -> 0
- net COL0: track 35.0 -> 75.7 mm
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- removed copper zone on B.Cu, net GND
Other:
- board outline removed

Commit message: Placed USB-C Components
Parts:
- removed F1: Polyfuse_Small, Fuse:Fuse_1206_3216Metric
- removed R3: 10k, Resistor_SMD:R_0805_2012Metric
- removed SW1: SW_Push, random-keyboard-parts:SKQG-1155865
- C1, C2, C3, C4, C5, C6, C7, F2, R1, R2, R4, R5, R6, R7, R8, R9, Y1: moved to B.Cu
- moved U1 117.0 mm to (145.4, 113.0), turned to 90 degrees
- moved C3 111.8 mm to (145.9, 120.8)
- moved C2 110.3 mm to (153.5, 118.0), turned to 90 degrees
- moved Y1 108.3 mm to (133.6, 113.3), turned to 270 degrees
- moved C5 108.0 mm to (133.6, 116.6)
- moved C6 103.2 mm to (136.8, 119.9), turned to 90 degrees
- moved R6 99.9 mm to (23.7, 37.5)
- moved C7 99.7 mm to (153.5, 108.5), turned to 270 degrees
- moved R4 96.6 mm to (155.6, 106.7), turned to 90 degrees
- moved C1 93.3 mm to (141.0, 105.2), turned to 180 degrees
- moved R5 92.3 mm to (23.7, 31.5)
- moved C4 92.3 mm to (133.6, 110.1), turned to 180 degrees
- moved R7 88.5 mm to (23.7, 43.6)
- moved R1 68.5 mm to (53.6, 42.2), turned to 90 degrees
- moved R8 68.5 mm to (47.2, 30.2), turned to 270 degrees
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Connections:
- U1 pad 1: Net-(U1-Pad1) -> COL7
- U1 pad 12: Net-(U1-Pad12) -> ROW4
- U1 pad 18: Net-(U1-Pad18) -> COL3
- U1 pad 19: Net-(U1-Pad19) -> COL2
- U1 pad 20: Net-(U1-Pad20) -> COL1
- U1 pad 21: Net-(U1-Pad21) -> COL0
- U1 pad 22: Net-(U1-Pad22) -> COL4
- U1 pad 26: Net-(U1-Pad26) -> LED_3
- U1 pad 27: Net-(U1-Pad27) -> LED_2
- U1 pad 28: Net-(U1-Pad28) -> LED_1
- U1 pad 29: Net-(U1-Pad29) -> ROW3
- U1 pad 30: Net-(U1-Pad30) -> ROW2
- U1 pad 31: Net-(U1-Pad31) -> ROW1
- U1 pad 32: Net-(U1-Pad32) -> ROW0
- U1 pad 36: Net-(U1-Pad36) -> COL5
- U1 pad 37: Net-(U1-Pad37) -> COL6
- U1 pad 38: Net-(U1-Pad38) -> COL8
- U1 pad 39: LED_3 -> COL9
- U1 pad 40: LED_2 -> COL10
- U1 pad 41: LED_1 -> COL11
Routing:
- net LED_1: track 0.00 -> 184.4 mm, vias 0 -> 2
- net LED_2: track 0.00 -> 178.2 mm, vias 0 -> 2
- net LED_3: track 0.00 -> 171.0 mm, vias 0 -> 2
- net COL0: track 75.7 -> 191.0 mm
- net COL11: track 54.4 -> 162.7 mm, vias 0 -> 1
- net COL10: track 54.4 -> 143.4 mm, vias 0 -> 1
- net COL1: track 75.7 -> 160.2 mm
- net COL2: track 75.7 -> 159.3 mm
- net GND: track 0.00 -> 81.4 mm
- net COL9: track 54.4 -> 123.2 mm, vias 0 -> 1
- net COL3: track 57.6 -> 124.8 mm, vias 0 -> 1
- net ROW0: track 95.2 -> 162.4 mm, vias 0 -> 2
- net +5V: track 0.00 -> 63.5 mm, vias 0 -> 4
- net COL5: track 57.6 -> 118.7 mm, vias 0 -> 3
- net COL8: track 36.3 -> 84.7 mm, vias 0 -> 1
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