File: V4N4G0RTH0N.kicad_pcb (KiCad board)
At the start: 2 copper layers, 242.9 x 96.6 mm, 123 parts, among them U1 ATmega32U4-A, U2 SRV05-4, Y1 16MHz

Commit message: V2
Parts:
- added D54: SOD-123, Diode_SMD:D_SOD-123, B.Cu at (122.6, 114.6)
- added F1: 500mA, Fuse:Fuse_0805_2012Metric, B.Cu at (56.6, 43.1)
Routing:
- net +5V: track 68.9 -> 212.7 mm, vias 6 -> 8
- net Net-(D54-Pad2): track 0.00 -> 24.9 mm
- net GND: track 275.7 -> 295.6 mm, vias 8 -> 10
- net VCC: track 16.1 -> 22.6 mm, vias 4 -> 5
Other:
- board text added: "S8erdude Designed"
- board text added: "Trashman Inspired"
- board text added: "V4N4G0RTH0N"
- board text removed: "V4N4G0RTH0N Trashman inspired S8erdude designed"

Commit message: Change silk
Parts:
- removed the G*** at (105.7, 77.3)
- added G***: LOGO, SILK:ORTHOVAN3, B.Cu at (198.8, 72.5)
- renumbered D54 to RESET
